File: einkbadge.kicad_pcb (KiCad board)
At the start: 2 copper layers, 0 parts

Commit message: update schematic
Parts:
- added BOOT1: BOOT, Package_SO:TS-1088-AR, F.Cu at (175.9, 86.2)
- added C1: 4.7u, Capacitor_SMD:C_0402_1005Metric, F.Cu at (174.2, 57.3)
- added C10: 100n, Capacitor_SMD:C_0402_1005Metric, F.Cu at (174.2, 71.0)
- added C100: 1uF, Capacitor_SMD:C_0402_1005Metric, F.Cu at (182.8, 57.3)
- added C101: 1uF, Capacitor_SMD:C_0402_1005Metric, F.Cu at (182.8, 59.2)
- added C102: 1uF, Capacitor_SMD:C_0402_1005Metric, F.Cu at (182.8, 61.2)
- added C103: 1uF, Capacitor_SMD:C_0402_1005Metric, F.Cu at (182.8, 63.2)
- added C104: 1uF, Capacitor_SMD:C_0402_1005Metric, F.Cu at (182.8, 65.1)
- added C105: 4.7uF, Capacitor_SMD:C_0603_1608Metric, F.Cu at (186.2, 67.2)
- added C106: 4.7uF, Capacitor_SMD:C_0603_1608Metric, F.Cu at (186.2, 69.7)
- added C107: 0.1uF, Capacitor_SMD:C_0402_1005Metric, F.Cu at (182.8, 67.1)
- added C108: 33pF, Capacitor_SMD:C_0402_1005Metric, F.Cu at (182.8, 69.1)
- added C11: 100n, Capacitor_SMD:C_0402_1005Metric, F.Cu at (177.1, 57.3)
- added C12: 100n, Capacitor_SMD:C_0402_1005Metric, F.Cu at (177.1, 59.2)
- added C13: 100n, Capacitor_SMD:C_0402_1005Metric, F.Cu at (177.1, 61.2)
- added C14: 100n, Capacitor_SMD:C_0402_1005Metric, F.Cu at (177.1, 63.2)
- added C15: 100n, Capacitor_SMD:C_0402_1005Metric, F.Cu at (177.1, 65.1)
- added C16: 100n, Capacitor_SMD:C_0402_1005Metric, F.Cu at (177.1, 67.1)
- added C17: 100n, Capacitor_SMD:C_0402_1005Metric, F.Cu at (177.1, 69.1)
- added C19: 15p, Capacitor_SMD:C_0402_1005Metric, F.Cu at (177.1, 71.0)
- added C2: 4.7u, Capacitor_SMD:C_0402_1005Metric, F.Cu at (174.2, 59.2)
- added C20: 15p, Capacitor_SMD:C_0402_1005Metric, F.Cu at (179.9, 57.3)
- added C22: 10u, Capacitor_SMD:C_0402_1005Metric, F.Cu at (179.9, 59.2)
- added C23: 10u, Capacitor_SMD:C_0402_1005Metric, F.Cu at (179.9, 61.2)
- added C3: 4.7u, Capacitor_SMD:C_0402_1005Metric, F.Cu at (174.2, 61.2)
- added C4: 10u, Capacitor_SMD:C_0805_2012Metric, F.Cu at (185.9, 116.8)
- added C5: 10u, Capacitor_SMD:C_0805_2012Metric, F.Cu at (185.9, 119.8)
- added C6: 100n, Capacitor_SMD:C_0402_1005Metric, F.Cu at (174.2, 63.2)
- added C7: 4.7u, Capacitor_SMD:C_0402_1005Metric, F.Cu at (174.2, 65.1)
- added C8: 100n, Capacitor_SMD:C_0402_1005Metric, F.Cu at (174.2, 67.1)
- added C9: 100n, Capacitor_SMD:C_0402_1005Metric, F.Cu at (174.2, 69.1)
- added C95: 1uF, Capacitor_SMD:C_0402_1005Metric, F.Cu at (179.9, 63.2)
- added C96: 1uF, Capacitor_SMD:C_0402_1005Metric, F.Cu at (179.9, 65.1)
- added C97: 1uF, Capacitor_SMD:C_0402_1005Metric, F.Cu at (179.9, 67.1)
- added C98: 1uF, Capacitor_SMD:C_0402_1005Metric, F.Cu at (179.9, 69.1)
- added C99: 1uF, Capacitor_SMD:C_0402_1005Metric, F.Cu at (179.9, 71.0)
- added D13: LED, LED_SMD:LED_0402_1005Metric, F.Cu at (186.1, 110.2)
- added D15: MBR0530, Diode_SMD:D_SOD-123, F.Cu at (175.7, 73.7)
- added D21: MBR0530, Diode_SMD:D_SOD-123, F.Cu at (175.7, 77.1)
- added D22: MBR0530, Diode_SMD:D_SOD-123, F.Cu at (175.7, 80.4)
- added D23: MBR0530, Diode_SMD:D_SOD-123, F.Cu at (175.7, 83.8)
- added H5: MountingHole, MountingHole:MountingHole_2.2mm_M2_Pad_Via, F.Cu at (175.7, 35.5)
- added H6: MountingHole, MountingHole:MountingHole_2.2mm_M2_Pad_Via, F.Cu at (175.7, 41.4)
- added H7: MountingHole, MountingHole:MountingHole_2.2mm_M2_Pad_Via, F.Cu at (175.7, 47.4)
- added H8: MountingHole, MountingHole:MountingHole_2.2mm_M2_Pad_Via, F.Cu at (175.7, 53.3)
- added J3: USB_C_Receptacle_USB2.0_14P, Connector_USB:USB_C_Receptacle_GCT_USB4105-xx-A_16P_TopMnt_Horizontal, F.Cu at (178.6, 110.6)
- added J4: Conn_01x03, Connector_PinHeader_1.00mm:PinHeader_1x03_P1.00mm_Vertical, F.Cu at (185.9, 62.4)
- added J6: lipo, Connector_JST:JST_PH_B2B-PH-K_1x02_P2.00mm_Vertical, F.Cu at (181.7, 51.0)
- added L1: 3.3u, Inductor_SMD:L_0805_2012Metric, F.Cu at (186.0, 122.7)
- added L6: 47uH 500mA, Inductor_SMD:L_APV_ANR4018, F.Cu at (184.3, 96.2)
- added Q1: AO3401A, Package_TO_SOT_SMD:SOT-23, F.Cu at (186.7, 82.8)
- added Q6: Si1308EDL, Package_TO_SOT_SMD:SOT-323_SC-70, F.Cu at (186.7, 107.4)
- added R29: 2.2R, Resistor_SMD:R_0402_1005Metric, F.Cu at (174.2, 94.4)
- added R30: 1M, Resistor_SMD:R_0402_1005Metric, F.Cu at (174.2, 96.4)
- added R31: 47, Resistor_SMD:R_0402_1005Metric, F.Cu at (174.2, 98.4)
- added R32: 10k, Resistor_SMD:R_0402_1005Metric, F.Cu at (174.2, 100.4)
- added R33: 33, Resistor_SMD:R_0402_1005Metric, F.Cu at (174.2, 102.3)
- added R34: 5.1k, Resistor_SMD:R_0402_1005Metric, F.Cu at (174.2, 104.3)
- added R35: 5.1k, Resistor_SMD:R_0402_1005Metric, F.Cu at (177.1, 94.4)
- added R36: 27, Resistor_SMD:R_0402_1005Metric, F.Cu at (177.1, 96.4)
- added R37: 27, Resistor_SMD:R_0402_1005Metric, F.Cu at (177.1, 98.4)
- added R38: 10k, Resistor_SMD:R_0402_1005Metric, F.Cu at (177.1, 100.4)
- added R39: 1.5k, Resistor_SMD:R_0402_1005Metric, F.Cu at (177.1, 102.3)
- added R40: 1k, Resistor_SMD:R_0402_1005Metric, F.Cu at (177.1, 104.3)
- added R41: 1K, Resistor_SMD:R_0402_1005Metric, F.Cu at (180.0, 94.4)
- added R42: 1k, Resistor_SMD:R_0402_1005Metric, F.Cu at (180.0, 96.4)
- added R43: 5.1k, Resistor_SMD:R_0402_1005Metric, F.Cu at (180.0, 98.4)
- added R44: 1.5k, Resistor_SMD:R_0402_1005Metric, F.Cu at (180.0, 100.4)
- added R45: 10k, Resistor_SMD:R_0402_1005Metric, F.Cu at (180.0, 102.3)
- added RESET1: RESET, Package_SO:TS-1088-AR, F.Cu at (182.2, 86.2)
- added SW21: SW_Push, Button_Switch_THT:SW_PUSH-12mm, F.Cu at (38.6, 126.0)
- added SW22: SW_Push, Button_Switch_THT:SW_PUSH-12mm, F.Cu at (103.2, 96.5)
- added SW23: SW_Push, Button_Switch_THT:SW_PUSH-12mm, F.Cu at (87.5, 111.3)
- added SW3: SW_Push, Button_Switch_THT:SW_PUSH-12mm, F.Cu at (38.6, 96.9)
- added SW4: SW_Push, Button_Switch_THT:SW_PUSH-12mm, F.Cu at (23.2, 111.4)
- added SW5: SW_SPDT, Package_SO:MST-12D18G3_SPDT, F.Cu at (178.3, 116.9)
- added SW7: SW_Push, Button_Switch_THT:SW_PUSH-12mm, F.Cu at (54.1, 111.5)
- added U11: SRV05-4, Package_TO_SOT_SMD:SOT-23-6, F.Cu at (186.8, 58.7)
- added U18: ST25DV04K-JFR6D3, Package_DFN_QFN:ST_UFDFPN-12-1EP_3x3mm_P0.5mm_EP1.4x2.55mm, F.Cu at (181.6, 82.9)
- added U5: RP2350_60QFN, Package_DFN_QFN:QFN-60-1EP_7x7mm_P0.4mm_EP3.4x3.4mm_ThermalVias, F.Cu at (183.3, 37.1)
- added U6: NCP1117-3.3_SOT223, Package_TO_SOT_SMD:SOT-223-3_TabPin2, F.Cu at (183.5, 76.2)
- added U9: TP4056-42-ESOP8, Package_SO:SOIC-8-1EP_3.9x4.9mm_P1.27mm_EP2.41x3.3mm_ThermalVias, F.Cu at (182.9, 45.1)
- added Y1: ABM8-272-T3, Crystal:Crystal_SMD_3225-4Pin_3.2x2.5mm, F.Cu at (184.1, 101.3)
Other:
- board outline added: 7.7 x 0.9 mm
