File: _autosave-einkbadge.kicad_pcb (KiCad board)
At the start: 2 copper layers, 108.2 x 99.1 mm, 427 parts, among them J1 USB_C_Receptacle_USB2.0_14P, J2 Conn_01x03, J3 Conn_01x14_Pin, J4 Conn_01x16_Pin, Q1 Si1308EDL, SW1 SW_Push, SW2 SW_Push, SW3 SW_Push, SW4 SW_Push, SW5 SW_Push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

Commit message: update
Parts:
- removed REF**112, REF**152, REF**232, REF**272, REF**312, REF**72: TestPoint_THTPad_D2.0mm_Drill1.0mm, TestPoint:TestPoint_THTPad_D2.0mm_Drill1.0mm
- added J5: Conn_01x03_Pin, Connector_PinHeader_2.54mm:PinHeader_1x03_P2.54mm_Vertical, F.Cu at (231.0, 125.5)
- added J6: Conn_01x03_Pin, Connector_PinHeader_2.54mm:PinHeader_1x03_P2.54mm_Vertical, F.Cu at (231.0, 135.6)
Routing:
- net +5V: track 20.0 -> 47.1 mm
- net +3V3: track 209.8 -> 224.1 mm, vias 4 -> 5
