File: _autosave-einkbadge.kicad_sch (KiCad schematic)
At the start: 79 parts, among them J1 USB_C_Receptacle_USB2.0_14P, J2 Conn_01x03, J3 Conn_01x14_Pin, J4 Conn_01x16_Pin, J5 Conn_01x03_Pin, J6 Conn_01x03_Pin, Q1 Si1308EDL, SW1 SW_Push, SW2 SW_Push, SW3 SW_Push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

Commit message: update
Parts:
- J5, J6: footprint (none) -> Connector_PinHeader_2.54mm:PinHeader_1x03_P2.54mm_Vertical
Changed lines of the file:
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@@
 			)
 		)
-		(property "Footprint" ""
+		(property "Footprint" "Connector_PinHeader_2.54mm:PinHeader_1x03_P2.54mm_Vertical"
 			(at 370.84 278.13 0)
 			(effects
@@
 			)
 		)
-		(property "Footprint" ""
+		(property "Footprint" "Connector_PinHeader_2.54mm:PinHeader_1x03_P2.54mm_Vertical"
 			(at 370.84 295.91 0)
 			(effects
